File: leguizamon/PROYECTO COMPLETO MOLLI.kicad_pcb (KiCad board)
At the start: 2 copper layers, 47 parts, among them J1 Conn_01x04_Pin, J11 Screw_Terminal_01x03, J12 Screw_Terminal_01x03, J13 Screw_Terminal_01x03, J14 Screw_Terminal_01x03, J15 Screw_Terminal_01x03, J16 Screw_Terminal_01x03, J17 Screw_Terminal_01x03, J2 Screw_Terminal_01x02, J3 Screw_Terminal_01x03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

Commit message: Add files via upload
6/6
Parts:
- added C3: 0.1, Capacitor_THT:C_Radial_D5.0mm_H5.0mm_P2.00mm, F.Cu at (71.3, 95.7)
- added R11: 1k, Resistor_SMD:R_0805_2012Metric, F.Cu at (78.4, 103.3)
- added R12: 1k, Resistor_SMD:R_0805_2012Metric, F.Cu at (78.4, 122.9)
- added R13: 1k, Resistor_SMD:R_0805_2012Metric, F.Cu at (78.4, 142.8)
- added R14: 1k, Resistor_SMD:R_0805_2012Metric, F.Cu at (78.4, 163.6)
- U5: footprint MacroLib:TO-220-3_Vertical -> Package_TO_SOT_SMD:TO-263-3_TabPin2
- U6: footprint EESTN5:ESP32_DEVKITC -> EESTN5:ESP32S
- moved D3 11.2 mm to (72.8, 142.8), turned to 0 degrees
- moved D5 11.2 mm to (72.8, 122.9), turned to 0 degrees
- moved D7 11.1 mm to (72.8, 103.3), turned to 0 degrees
- moved D2 11.1 mm to (72.8, 163.6), turned to 0 degrees
- moved U5 7.13 mm to (47.3, 106.4), turned to 0 degrees
- moved J2 5.27 mm to (57.6, 98.4)
- moved R10 2.81 mm to (54.6, 139.4)
- moved R9 2.57 mm to (47.0, 134.1)
- moved C1 1.27 mm to (35.0, 103.9)
- moved C2 1.27 mm to (35.0, 109.0)
Connections:
- U1 pad 2: Net-(D2-A) -> GND
- U2 pad 2: Net-(D3-A) -> GND
- U3 pad 2: Net-(D5-A) -> GND
- U4 pad 2: Net-(D7-A) -> GND
Routing:
- net +12V: track 311.7 -> 318.1 mm
- net GND: track 3.24 -> 0.01 mm
- net D echo: track 36.1 -> 33.0 mm
- net +5V: track 32.4 -> 29.4 mm
- net DATO K2: track 8.76 -> 11.3 mm
- net Net-(D8-A): track 18.9 -> 16.4 mm
- net Net-(D4-A): track 18.5 -> 16.2 mm
- net Net-(D6-A): track 18.6 -> 16.3 mm
- net echo: track 5.31 -> 3.65 mm
- net Net-(D2-A): track 2.31 -> 3.80 mm
- net Net-(D7-A): track 2.32 -> 3.80 mm
- net Net-(D5-A): track 2.33 -> 3.80 mm
- net Net-(D3-A): track 2.41 -> 3.80 mm
- net DATO K4: track 35.0 -> 36.2 mm
- net DATO K3: track 17.9 -> 19.1 mm
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
Commit message: Add files via upload
arregle
Parts:
- C3: moved to B.Cu
- D1, D4, D6, D8: footprint Diode_SMD:D_0805_2012Metric -> Diode_SMD:D_SMA
- Q1, Q2, Q3, Q4: value BF457 -> MMBT2222A
- moved Q4 64.2 mm to (86.5, 172.8), turned to 90 degrees
- moved Q1 56.1 mm to (86.5, 112.7), turned to 90 degrees
- moved Q3 24.0 mm to (86.5, 152.2), turned to 90 degrees
- moved Q2 15.8 mm to (86.5, 132.4), turned to 90 degrees
- moved R6 5.42 mm to (76.3, 133.3)
- moved R4 5.40 mm to (76.3, 153.2)
- moved R8 5.39 mm to (76.3, 113.7)
- moved R2 5.32 mm to (76.3, 173.7)
- moved C3 4.40 mm to (70.9, 100.1), turned to 180 degrees
- moved J2 2.49 mm to (57.6, 100.8)
- moved D8 1.15 mm to (81.4, 107.5)
- moved D1 1.06 mm to (81.3, 167.6)
- moved D4 1.06 mm to (81.3, 146.9)
- moved D6 1.06 mm to (81.3, 127.1)
- moved R11 0.09 mm to (78.5, 103.3)
Connections:
- Q1 pad 1: GND -> Net-(Q1-B)
- Q1 pad 2: Net-(D1-A) -> GND
- Q1 pad 3: Net-(Q1-B) -> Net-(D8-A)
- Q2 pad 1: GND -> Net-(Q2-B)
- Q2 pad 2: Net-(D4-A) -> GND
- Q2 pad 3: Net-(Q2-B) -> Net-(D6-A)
- Q3 pad 1: GND -> Net-(Q3-B)
- Q3 pad 2: Net-(D6-A) -> GND
- Q3 pad 3: Net-(Q3-B) -> Net-(D4-A)
- Q4 pad 1: GND -> Net-(Q4-B)
- Q4 pad 2: Net-(D8-A) -> GND
- Q4 pad 3: Net-(Q4-B) -> Net-(D1-A)
- R2 pad 2: Net-(Q1-B) -> Net-(Q4-B)
- R4 pad 2: Net-(Q2-B) -> Net-(Q3-B)
- R6 pad 2: Net-(Q3-B) -> Net-(Q2-B)
- R8 pad 2: Net-(Q4-B) -> Net-(Q1-B)
Routing:
- net Net-(Q4-B): track 4.02 -> 8.34 mm
- net Net-(Q1-B): track 4.02 -> 8.34 mm
- net Net-(Q2-B): track 4.02 -> 8.32 mm
- net Net-(Q3-B): track 4.02 -> 8.32 mm
- net Net-(D4-A): track 16.2 -> 18.3 mm
- net Net-(D8-A): track 16.4 -> 18.5 mm
- net Net-(D6-A): track 16.3 -> 18.4 mm
- net Net-(D1-A): track 18.0 -> 19.9 mm
