File: leguizamon/PROYECTO COMPLETO MOLLI.kicad_sch (KiCad schematic)
At the start: 47 parts, among them J1 Conn_01x04_Pin, J11 Screw_Terminal_01x03, J12 Screw_Terminal_01x03, J13 Screw_Terminal_01x03, J14 Screw_Terminal_01x03, J15 Screw_Terminal_01x03, J16 Screw_Terminal_01x03, J17 Screw_Terminal_01x03, J2 Screw_Terminal_01x02, J3 Screw_Terminal_01x03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

Commit message: Add files via upload
6/6
Parts:
- added C3: 0.1, Capacitor_THT:C_Radial_D5.0mm_H5.0mm_P2.00mm, symbol Device:C
- added R11, R12, R13, R14: 1k, Resistor_SMD:R_0805_2012Metric, symbol Device:R
- U5: footprint MacroLib:TO-220-3_Vertical -> Package_TO_SOT_SMD:TO-263-3_TabPin2
- U6: footprint EESTN5:ESP32_DEVKITC -> EESTN5:ESP32S
Connections:
- net +12V: now also C3.1, R11.2, R12.2, R13.2, R14.2
- net GND: now also U1.2, U2.2, U3.2, U4.2, C3.2
- net at D5.2 (A): now also R12.1; no longer U3.2
- net at D2.2 (A): now also R14.1; no longer U1.2
- net at D7.2 (A): now also R11.1; no longer U4.2
- net at D3.2 (A): now also R13.1; no longer U2.2
Other:
- moved on the sheet: D2, D3, D5, D7, R10, R9, U6

Commit message: Add files via upload
arregle
Parts:
- removed Q1, Q2, Q3, Q4: BF457, Package_TO_SOT_SMD:SOT-23, symbol Transistor_BJT:BF457
- added Q1, Q2, Q3, Q4: MMBT2222A, Package_TO_SOT_SMD:SOT-23, symbol Transistor_BJT:MMBT2222A
- D1, D4, D6, D8: footprint Diode_SMD:D_0805_2012Metric -> Diode_SMD:D_SMA
Connections:
- net GND: now also Q1.2 (E), Q2.2 (E), Q3.2 (E), Q4.2 (E)
- net at D6.2 (A), K3.A2: now also Q2.3 (C)
- net at R6.2: now also Q2.1 (B)
- net at D1.2 (A), K1.A2: now also Q4.3 (C)
- net at R2.2: now also Q4.1 (B)
- net at D4.2 (A), K2.A2: now also Q3.3 (C)
- net at D8.2 (A), K4.A2: now also Q1.3 (C)
- net at R4.2: now also Q3.1 (B)
- net at R8.2: now also Q1.1 (B)
